File: hardware/main_pcb_hw5/main_pcb_hw5.kicad_pcb (KiCad board)
At the start: 2 copper layers, 100 x 100 mm, 31 parts, among them J1 MEGA BOTTOM, J10 GBA_Slot, J3 CART SLOT TOP ROW, J4 CART SLOT FRONT ROW, J6 5V USB, J7 Conn_01x07, J8 EXP2, J9 EXP1, M2_1 Screw_Terminal_01x01, M2_2 Screw_Terminal_01x01, M2_3 Screw_Terminal_01x01, M2_4 Screw_Terminal_01x01, M2_5 Screw_Terminal_01x01, M2_6 Screw_Terminal_01x01, M2_7 Screw_Terminal_01x01, M2_8 Screw_Terminal_01x01, M2_9 Screw_Terminal_01x01, SW1 VOLTAGE, SW2 POWER, U1 TPS2113PW, U2 DS3231MZ

Commit message: cliche commit summary goes here
Parts:
- removed the G*** at (150.0, 62.5)
- removed M2_5, M2_6, M2_7, M2_8, M2_9: Screw_Terminal_01x01, MountingHole:MountingHole_2.2mm_M2_ISO7380_Pad
- added C10: 10uF, Capacitor_SMD:C_0805_2012Metric, F.Cu at (145.2, 171.7)
- added C11: 10uF, Capacitor_SMD:C_0805_2012Metric, F.Cu at (140.9, 174.6)
- added C12: 1uF, Capacitor_SMD:C_0805_2012Metric, F.Cu at (38.8, 186.5)
- added C13: 100nF, Capacitor_SMD:C_0805_2012Metric, B.Cu at (99.4, 184.5)
- added C14: 1uF, Capacitor_SMD:C_0805_2012Metric, F.Cu at (66.2, 182.5)
- added C15: 100nf, Capacitor_SMD:C_0805_2012Metric, B.Cu at (33.4, 170.8)
- added C16: 100nF, Capacitor_SMD:C_0805_2012Metric, B.Cu at (77.3, 184.4)
- added C17: 100nf, Capacitor_SMD:C_0805_2012Metric, B.Cu at (29.9, 170.8)
- added C18: 1uF, Capacitor_SMD:C_0805_2012Metric, F.Cu at (115.1, 182.6)
- added C19: 100nF, Capacitor_SMD:C_0805_2012Metric, B.Cu at (31.5, 183.9)
- added C20: 1uF, Capacitor_SMD:C_0805_2012Metric, F.Cu at (89.1, 182.3)
- added C21: 100nF, Capacitor_SMD:C_0805_2012Metric, B.Cu at (121.8, 184.2)
- added C22: 1uF, Capacitor_SMD:C_0805_2012Metric, F.Cu at (47.5, 182.6)
- added C23: 0.1u, Capacitor_SMD:C_0805_2012Metric, F.Cu at (75.0, 138.9)
- added C24: 100nF, Capacitor_SMD:C_0805_2012Metric, B.Cu at (144.6, 184.2)
- added C25: 10uf, Capacitor_SMD:C_0805_2012Metric, F.Cu at (78.3, 155.6)
- added C26: 10uf, Capacitor_SMD:C_0805_2012Metric, F.Cu at (85.4, 154.4)
- added C27: 0.1u, Capacitor_SMD:C_0805_2012Metric, F.Cu at (74.9, 141.0)
- added C28: 100nF, Capacitor_SMD:C_0805_2012Metric, F.Cu at (129.6, 133.7)
- added C29: 100nF, Capacitor_SMD:C_0805_2012Metric, F.Cu at (129.8, 131.4)
- added C30: 1uF, Capacitor_SMD:C_0805_2012Metric, F.Cu at (137.5, 182.4)
- added C31: 100nF, Capacitor_SMD:C_0805_2012Metric, B.Cu at (54.2, 183.9)
- added C34: 10u, Capacitor_SMD:C_0805_2012Metric, F.Cu at (71.5, 138.9)
- added C35: 22uf, Capacitor_SMD:C_0805_2012Metric, F.Cu at (120.3, 179.8)
- added C36: 470u, Capacitor_Tantalum_SMD:CP_EIA-7343-31_Kemet-D, F.Cu at (81.0, 144.7)
- added C37: 22uf, Capacitor_SMD:C_0805_2012Metric, F.Cu at (123.9, 179.8)
- added C38: 0.1u, Capacitor_SMD:C_0805_2012Metric, F.Cu at (110.6, 166.8)
- added C39: C_Small_0.1uf, Capacitor_SMD:C_0805_2012Metric, F.Cu at (106.3, 182.2)
- added C6: 10uF, Capacitor_SMD:C_0805_2012Metric, F.Cu at (131.5, 160.4)
- added C7: 100nF, Capacitor_SMD:C_0805_2012Metric, F.Cu at (130.9, 169.5)
- added C8: 10uF, Capacitor_SMD:C_0805_2012Metric, F.Cu at (81.8, 171.6)
- added C9: 10uF, Capacitor_SMD:C_0805_2012Metric, F.Cu at (78.3, 171.6)
- added Card1: TF PUSH, !MiniReader:TF-SMD_TF-PUSH, F.Cu at (113.0, 145.1)
- added D10: SK6812MINI, !MiniReader:LED_SK6812MINI_PLCC4_3.5x3.5mm_P1.75mm, B.Cu at (228.8, 164.8)
- added D11: 1N4148W, Diode_SMD:D_SOD-123, F.Cu at (87.1, 116.3)
- added D12: SK6812MINI, !MiniReader:LED_SK6812MINI_PLCC4_3.5x3.5mm_P1.75mm, B.Cu at (235.3, 158.7)
- added D13: 1N4148W, Diode_SMD:D_SOD-123, F.Cu at (84.7, 116.4)
- added D14: 1N4148W, Diode_SMD:D_SOD-123, F.Cu at (89.7, 116.3)
- added D15: SK6812MINI, !MiniReader:LED_SK6812MINI_PLCC4_3.5x3.5mm_P1.75mm, B.Cu at (223.0, 154.8)
- added D16: 1N4148W, Diode_SMD:D_SOD-123, F.Cu at (77.2, 116.4)
- added D17: SK6812MINI, !MiniReader:LED_SK6812MINI_PLCC4_3.5x3.5mm_P1.75mm, B.Cu at (223.0, 158.1)
- added D18: 1N4148W, Diode_SMD:D_SOD-123, F.Cu at (80.4, 121.5)
- added D19: SK6812MINI, !MiniReader:LED_SK6812MINI_PLCC4_3.5x3.5mm_P1.75mm, B.Cu at (223.0, 161.5)
- added D2: 1N4148W, Diode_SMD:D_SOD-123, F.Cu at (102.1, 116.3)
- added D20: 1N4148W, Diode_SMD:D_SOD-123, F.Cu at (83.2, 121.5)
- added D21: 1N4148W, Diode_SMD:D_SOD-123, F.Cu at (99.6, 116.3)
- added D22: SK6812MINI, !MiniReader:LED_SK6812MINI_PLCC4_3.5x3.5mm_P1.75mm, B.Cu at (217.2, 148.1)
- added D23: 1N4148W, Diode_SMD:D_SOD-123, F.Cu at (85.8, 121.5)
- added D24: SK6812MINI, !MiniReader:LED_SK6812MINI_PLCC4_3.5x3.5mm_P1.75mm, B.Cu at (217.2, 151.4)
- added D25: 1N4148W, Diode_SMD:D_SOD-123, F.Cu at (90.9, 121.5)
- added D26: 1N4148W, Diode_SMD:D_SOD-123, F.Cu at (92.1, 116.3)
- added D27: SK6812MINI, !MiniReader:LED_SK6812MINI_PLCC4_3.5x3.5mm_P1.75mm, B.Cu at (235.4, 153.7)
- added D28: SK6812MINI, !MiniReader:LED_SK6812MINI_PLCC4_3.5x3.5mm_P1.75mm, B.Cu at (217.2, 158.1)
- added D29: 1N4148W, Diode_SMD:D_SOD-123, F.Cu at (88.5, 121.5)
- added D3: 1N4148W, Diode_SMD:D_SOD-123, F.Cu at (93.3, 121.5)
- added D31: 1N4148W, Diode_SMD:D_SOD-123, F.Cu at (97.0, 116.3)
- added D33: 1N4148W, Diode_SMD:D_SOD-123, F.Cu at (98.5, 121.5)
- added D4: 1N4148W, Diode_SMD:D_SOD-123, F.Cu at (95.8, 121.5)
- added D5: SK6812MINI, !MiniReader:LED_SK6812MINI_PLCC4_3.5x3.5mm_P1.75mm, B.Cu at (228.8, 154.8)
- added D6: SK6812MINI, !MiniReader:LED_SK6812MINI_PLCC4_3.5x3.5mm_P1.75mm, B.Cu at (228.8, 158.1)
- added D7: 1N4148W, Diode_SMD:D_SOD-123, F.Cu at (79.7, 116.4)
- added D8: SK6812MINI, !MiniReader:LED_SK6812MINI_PLCC4_3.5x3.5mm_P1.75mm, B.Cu at (228.8, 161.5)
- added D9: 1N4148W, Diode_SMD:D_SOD-123, F.Cu at (82.2, 116.4)
- added F1: MF-NSMF150-2, Fuse:Fuse_1206_3216Metric, B.Cu at (29.5, 167.4)
- added G***: LOGO, LOGO, F.Cu at (150.3, 162.3)
- added G***: LOGO, LOGO, F.Cu at (150.3, 169.2)
- added J11: SHOUHANTYPE-C16PIN2MD-073, !MiniReader:USB-C-SMD_TYPE-C-6PIN-2MD-073, F.Cu at (144.4, 184.5)
- added J12: SHOUHANTYPE-C16PIN2MD-073, !MiniReader:USB-C-SMD_TYPE-C-6PIN-2MD-073, F.Cu at (121.9, 184.5)
- added J14: Conn_01x09, Connector_PinHeader_1.00mm:PinHeader_1x09_P1.00mm_Vertical, F.Cu at (22.9, 141.3)
- added J2: MEGA BOTTOM, !MiniReader:MEGA2560_PRO_EMBED_SMD, F.Cu at (49.4, 145.1)
- added J5: Conn_01x05, Connector_PinHeader_1.00mm:PinHeader_1x05_P1.00mm_Vertical, F.Cu at (84.9, 148.3)
- added JP1: Jumper_2_Open, Jumper:SolderJumper-2_P1.3mm_Open_TrianglePad1.0x1.5mm, B.Cu at (234.8, 163.4)
- added L1: 60R@100MHz, Inductor_SMD:L_1206_3216Metric, B.Cu at (32.0, 167.5)
- added R10: 10K, Resistor_SMD:R_0805_2012Metric, F.Cu at (101.5, 180.2)
- added R11: 10K, Resistor_SMD:R_0805_2012Metric, F.Cu at (128.6, 185.0)
- added R12: 10K, Resistor_SMD:R_0805_2012Metric, F.Cu at (128.8, 182.9)
- added R13: 10K, Resistor_SMD:R_0805_2012Metric, F.Cu at (151.4, 184.4)
- added R14: 10K, Resistor_SMD:R_0805_2012Metric, F.Cu at (151.4, 182.4)
- added R15: 3.3K, Resistor_SMD:R_0805_2012Metric, F.Cu at (92.1, 143.5)
- added R16: 3.3K, Resistor_SMD:R_0805_2012Metric, F.Cu at (95.1, 143.5)
- added R17: 3.3K, Resistor_SMD:R_0805_2012Metric, F.Cu at (98.0, 143.5)
- added R18: 3.3K, Resistor_SMD:R_0805_2012Metric, F.Cu at (101.0, 143.5)
- added R3: 10K, Resistor_SMD:R_0805_2012Metric, F.Cu at (24.0, 184.3)
- added R4: 10K, Resistor_SMD:R_0805_2012Metric, F.Cu at (24.1, 182.4)
- added R5: 10K, Resistor_SMD:R_0805_2012Metric, F.Cu at (38.9, 184.4)
- added R6: 10K, Resistor_SMD:R_0805_2012Metric, F.Cu at (42.4, 182.5)
- added R7: 10K, Resistor_SMD:R_0805_2012Metric, F.Cu at (83.8, 182.4)
- added R8: 10K, Resistor_SMD:R_0805_2012Metric, F.Cu at (69.6, 182.4)
- added R9: 10K, Resistor_SMD:R_0805_2012Metric, F.Cu at (92.5, 182.2)
- added SW10: SKQGABE010, !MiniReader:SW-SMD_4P-L4.5-W4.5-P3.00-LS6.8, B.Cu at (98.0, 120.3)
- added SW11: b, MX_Hotswap:MX-Hotswap-1U, B.Cu at (132.5, 149.2)
- added SW12: SKQGABE010, !MiniReader:SW-SMD_4P-L4.5-W4.5-P3.00-LS6.8, B.Cu at (81.0, 141.8)
- added SW13: c, MX_Hotswap:MX-Hotswap-1U, B.Cu at (115.9, 131.4)
- added SW14: SKQGABE010, !MiniReader:SW-SMD_4P-L4.5-W4.5-P3.00-LS6.8, B.Cu at (80.8, 120.4)
- added SW15: d, MX_Hotswap:MX-Hotswap-1U, B.Cu at (133.1, 117.1)
- added SW16: SKQGABE010, !MiniReader:SW-SMD_4P-L4.5-W4.5-P3.00-LS6.8, B.Cu at (98.0, 141.7)
- added SW17: l1, MX_Hotswap:MX-Hotswap-1U, B.Cu at (-89.3, 73.2)
- added SW19: r1, MX_Hotswap:MX-Hotswap-1U, B.Cu at (-6.45, 71.1)
- added SW21: SKQGABE010, !MiniReader:SW-SMD_4P-L4.5-W4.5-P3.00-LS6.8, B.Cu at (149.7, 176.7)
- added SW22: Rotary_Encoder_Switch, !MiniReader:RotaryEncoder_EC11_no_mp, B.Cu at (89.1, 129.6)
- added SW3: down, MX_Hotswap:MX-Hotswap-1U, B.Cu at (46.8, 148.9)
- added SW4: l2l, MX_Hotswap:MX-Hotswap-1U, B.Cu at (-31.5, 94.5)
- added SW5: left, MX_Hotswap:MX-Hotswap-1U, B.Cu at (31.5, 132.6)
- added SW6: r2h, MX_Hotswap:MX-Hotswap-1U, B.Cu at (-53.9, 112.5)
- added SW7: right, MX_Hotswap:MX-Hotswap-1U, B.Cu at (61.8, 133.1)
- added SW8: r2l, MX_Hotswap:MX-Hotswap-1U, B.Cu at (-35.0, 114.2)
- added SW9: a, MX_Hotswap:MX-Hotswap-1U, B.Cu at (148.6, 130.3)
- added U10: UZ1085L-33-TN3-R, Package_TO_SOT_SMD:TO-252-2, F.Cu at (125.0, 175.3)
- added U11: DS1307DTR(XBLW), Package_SO:SOIC-8_3.9x4.9mm_P1.27mm, F.Cu at (109.1, 161.2)
- added U12: snesCIC PIC12F629T-E/MF1, Package_DFN_QFN:DFN-8-1EP_4x4mm_P0.8mm_EP2.39x2.21mm, F.Cu at (105.7, 178.9)
- added U13: 74LVC125APW,118, !MiniReader:TSSOP-14_L5.0-W4.4-P0.65-LS6.4-BL, F.Cu at (101.3, 150.3)
- added U3: SL2.1A, Package_SO:SOIC-16_4.55x10.3mm_P1.27mm, F.Cu at (148.2, 177.0)
- added U4: SMAJ8.0CA-TP, Diode_SMD:D_SMA, B.Cu at (31.7, 174.0)
- added U5: SMAJ8.0CA-TP, Diode_SMD:D_SMA, F.Cu at (92.0, 152.6)
- added U6: SMAJ8.0CA-TP, Diode_SMD:D_SMA, F.Cu at (92.1, 149.0)
- added U7: SMAJ8.0CA-TP, Diode_SMD:D_SMA, F.Cu at (80.1, 152.7)
- added U8: SMAJ8.0CA-TP, Diode_SMD:D_SMA, F.Cu at (80.1, 149.1)
- added U9: TPS2113PW, Package_SO:TSSOP-8_4.4x3mm_P0.65mm, F.Cu at (72.9, 136.0)
- added Y1: 12mhz, Crystal:Crystal_HC49-4H_Vertical, F.Cu at (91.2, 178.3)
- added Y2: 12mhz, Crystal:Crystal_HC49-4H_Vertical, F.Cu at (134.2, 178.5)
- added Y3: 32.768mhz, Crystal:Crystal_HC49-4H_Vertical, F.Cu at (110.0, 171.5)
- BT1: moved to F.Cu
- C1: value 470u -> 100nF; footprint Capacitor_THT:CP_Radial_D8.0mm_P3.50mm -> Capacitor_SMD:C_0805_2012Metric
- C2, C3, C5: value 0.1u -> 100nF; footprint Capacitor_SMD:C_0402_1005Metric_Pad0.74x0.62mm_HandSolder -> Capacitor_SMD:C_0805_2012Metric
- C4: value 10u -> 100nF; footprint Capacitor_SMD:C_0402_1005Metric_Pad0.74x0.62mm_HandSolder -> Capacitor_SMD:C_0805_2012Metric
- D1: value LED -> 1N4148W; footprint LED_THT:LED_D3.0mm -> Diode_SMD:D_SOD-123
- J1: value MEGA BOTTOM -> Conn_01x03_Female; footprint !OSCR:MEGA2560_PRO_MINI -> Connector_PinSocket_2.54mm:PinSocket_1x03_P2.54mm_Vertical; moved to B.Cu
- J10: value GBA_Slot -> SHOUHANTYPE-C16PIN2MD-073; footprint !sanni:GBA-SLOT-B -> !MiniReader:USB-C-SMD_TYPE-C-6PIN-2MD-073
- J3: value CART SLOT TOP ROW -> Conn_02x36; footprint !OSCR:Cartridge_Port_Adapter-Back -> !MiniReader:Secondary_Board_Connector
- J4: value CART SLOT FRONT ROW -> 5V USB; footprint !OSCR:Cartridge_Port_Adapter-Front -> TestPoint:TestPoint_Pad_D2.0mm
- J6: value 5V USB -> Conn_01x05; footprint Connector_PinHeader_2.54mm:PinHeader_1x01_P2.54mm_Vertical -> Connector_PinHeader_1.00mm:PinHeader_1x05_P1.00mm_Vertical
- J7: value Conn_01x07 -> SHOUHANTYPE-C16PIN2MD-073; footprint !OSCR:Clock_Generator_Header -> !MiniReader:USB-C-SMD_TYPE-C-6PIN-2MD-073
- J8: value EXP2 -> SHOUHANTYPE-C16PIN2MD-073; footprint !OSCR:LCD_Header -> !MiniReader:USB-C-SMD_TYPE-C-6PIN-2MD-073
- J9: value EXP1 -> SHOUHANTYPE-C16PIN2MD-073; footprint !OSCR:LCD_Header -> !MiniReader:USB-C-SMD_TYPE-C-6PIN-2MD-073
- M2_1, M2_3: moved to B.Cu
- R1: value 220R -> 10k; footprint Resistor_THT:R_Axial_DIN0207_L6.3mm_D2.5mm_P10.16mm_Horizontal -> Resistor_SMD:R_0805_2012Metric; moved to B.Cu
- R2: footprint Resistor_SMD:R_0402_1005Metric_Pad0.72x0.64mm_HandSolder -> Resistor_SMD:R_0805_2012Metric
- SW1: value VOLTAGE -> up; footprint !OSCR:Power_Switch -> MX_Hotswap:MX-Hotswap-1U; moved to B.Cu
- SW2: value POWER -> l2h; footprint !OSCR:Power_Switch -> MX_Hotswap:MX-Hotswap-1U; moved to B.Cu
- U1: value TPS2113PW -> STM32F072CBT6; footprint Personal:Texas_Instruments-TPS2113PW-Level_A -> Package_QFP:LQFP-48_7x7mm_P0.5mm
- U2: value DS3231MZ -> SL2.1A; footprint Package_SO:SOIC-8_3.9x4.9mm_P1.27mm -> Package_SO:SOIC-16_4.55x10.3mm_P1.27mm
- moved SW2 256.2 mm to (-56.3, 94.4), turned to 180 degrees
- moved M2_3 205.4 mm to (24.4, 187.6)
- moved J7 152.5 mm to (31.9, 184.5), turned to 0 degrees
- moved SW1 150.3 mm to (47.2, 114.2), turned to 180 degrees
- moved M2_1 150.3 mm to (-4.72, 157.3)
- moved BT1 136.8 mm to (97.5, 166.9), turned to 0 degrees
- moved J10 126.5 mm to (99.4, 184.5), turned to 0 degrees
- moved J8 125.3 mm to (54.5, 184.5), turned to 0 degrees
- moved J9 124.1 mm to (76.9, 184.5), turned to 0 degrees
- moved J3 118.6 mm to (54.4, 189.7), turned to 0 degrees
- moved R2 117.8 mm to (71.5, 141.0)
- moved U2 104.2 mm to (81.9, 177.0), turned to 90 degrees
- moved J1 103.2 mm to (214.9, 168.6), turned to -90 degrees
- moved J4 100.5 mm to (25.3, 165.2), turned to 0 degrees
- moved C1 96.9 mm to (121.0, 169.4)
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Connections:
- C1 pad 1: VCC -> +3V3
- C2 pad 1: GND -> +3V3
- C2 pad 2: +3V3 -> GND
- C3 pad 1: +5V -> +3V3
- C4 pad 1: VCC -> +3V3
- C5 pad 1: VBUS -> +3V3
- D1 pad 2: VCC -> A8
- J1 pad 1: D30 -> GND
- J1 pad 2: D31 -> Net-(D5-DOUT)
- J1 pad 3: D28 -> +5V
- J10 pad 1: VCC -> GND
- J10 pad 10: A4 -> Net-(J10-CC2)
- J10 pad 11: A5 -> +5V
- J10 pad 12: A6 -> GND
- J10 pad 13: A7 -> GND
- J10 pad 14: A8 -> GND
- J10 pad 2: D16 -> +5V
- J10 pad 3: D8 -> unconnected-(J10-SBU2-Pad3)
- J10 pad 4: D9 -> Net-(J10-CC1)
- J10 pad 5: D6 -> /D4+
- J10 pad 6: A0 -> /D4+
- J10 pad 7: A1 -> /D4+
- J10 pad 8: A2 -> /D4+
- J10 pad 9: A3 -> unconnected-(J10-SBU1-Pad9)
- J3 pad 1: VCC -> CLK1
- J3 pad 10: A6 -> A13
- J3 pad 11: A7 -> A12
- J3 pad 12: A8 -> A11
- J3 pad 13: A9 -> A10
- J3 pad 14: A10 -> A9
- J3 pad 15: A11 -> A8
- J3 pad 16: A12 -> A1
- J3 pad 17: A13 -> D8
- J3 pad 18: A14 -> D7
- J3 pad 19: A15 -> D6
- J3 pad 2: unconnected-(J3-Pin_2-Pad2) -> D15
- J3 pad 20: D37 -> D16
- J3 pad 21: D36 -> D17
- J3 pad 22: D35 -> A2
- J3 pad 23: D34 -> A3
- J3 pad 24: D33 -> A4
- J3 pad 25: D32 -> D42
- J3 pad 26: D31 -> D22
- J3 pad 27: D30 -> D23
- J3 pad 28: D17 -> D25
- J3 pad 29: D16 -> D24
- J3 pad 3: unconnected-(J3-Pin_3-Pad3) -> D14
- J3 pad 30: D6 -> D26
- J3 pad 31: D7 -> D27
- J3 pad 32: D8 -> A15
- J3 pad 33: D9 -> A14
- J3 pad 34: D53 -> A13
- J3 pad 35: D52 -> A12
- J3 pad 36: D51 -> D3
- J3 pad 37: D50 -> D40
- J3 pad 38: GND -> D41
- J3 pad 4: A0 -> D29
- J3 pad 5: A1 -> CLK0
- J3 pad 6: A2 -> A0
- J3 pad 7: A3 -> D28
- J3 pad 8: A4 -> A15
- J3 pad 9: A5 -> A14
- J4 pad 1: GND -> +5.0V
- J6 pad 1: VBUS -> GND
- J7 pad 1: VCC -> GND
- J7 pad 2: GND -> +5V
- J7 pad 3: D20 -> unconnected-(J7-SBU2-Pad3)
- J7 pad 4: D21 -> Net-(J7-CC1)
- J7 pad 5: CLK2 -> /D1+
- J7 pad 6: CLK1 -> /D1+
- J7 pad 7: CLK0 -> /D1-
- J8 pad 1: +3V3 -> GND
- J8 pad 10: D50 -> Net-(J8-CC2)
- J8 pad 2: GND -> +5V
- J8 pad 3: RESET -> unconnected-(J8-SBU2-Pad3)
- J8 pad 4: unconnected-(J8-Pin_4-Pad4) -> Net-(J8-CC1)
- J8 pad 5: D51 -> /D2+
- J8 pad 6: D19 -> /D2+
- J8 pad 7: D53 -> /D2+
- J8 pad 8: D18 -> /D2+
- J8 pad 9: D52 -> unconnected-(J8-SBU1-Pad9)
- J9 pad 1: +5V -> GND
- J9 pad 10: unconnected-(J9-Pin_10-Pad10) -> Net-(J9-CC2)
- J9 pad 2: GND -> +5V
- J9 pad 4: unconnected-(J9-Pin_4-Pad4) -> Net-(J9-CC1)
- J9 pad 5: D13 -> /D3+
- J9 pad 6: D10 -> /D3+
- J9 pad 7: D11 -> /D3+
- J9 pad 8: D12 -> /D3+
- J9 pad 9: D39 -> unconnected-(J9-SBU1-Pad9)
- R1 pad 1: Net-(D1-K) -> BOOT0
- R1 pad 2: D38 -> GND
- R2 pad 2: Net-(U1-ILIM) -> Net-(U9-ILIM)
- SW1 pad 1: +3V3 -> Net-(D1-K)
- SW1 pad 2: VCC -> col0
- SW2 pad 1: VBUS -> Net-(D2-K)
- SW2 pad 2: +5V -> col0
- U1 pad 1: unconnected-(U1-STAT-Pad1) -> +3V3
- U1 pad 2: GND -> col5
- U1 pad 3: D38 -> col6
- U1 pad 4: Net-(U1-ILIM) -> col7
- U1 pad 5: GND -> col8
- U1 pad 6: +5V -> col9
- U1 pad 7: VCC -> NRST
- U1 pad 8: +3V3 -> GND
- U2 pad 1: unconnected-(U2-32KHZ-Pad1) -> /D4+
- U2 pad 2: VBUS -> /D4+
- U2 pad 3: unconnected-(U2-~{INT}/SQW-Pad3) -> /D3+
- U2 pad 4: unconnected-(U2-~{RST}-Pad4) -> /D3+
- U2 pad 5: GND -> /D2+
- U2 pad 6: +BATT -> /D2+
- U2 pad 7: D20 -> /D1-
- U2 pad 8: D21 -> /D1+
Routing:
- net GND: track 382.8 -> 0.00 mm, vias 215 -> 0
- net VCC: track 282.8 -> 0.00 mm, vias 2 -> 0
- net D16: track 160.1 -> 0.00 mm, vias 1 -> 0
- net D8: track 149.5 -> 0.00 mm, vias 3 -> 0
- net D9: track 136.0 -> 0.00 mm, vias 2 -> 0
- net RESET: track 134.1 -> 0.00 mm, vias 1 -> 0
- net A14: track 127.6 -> 0.00 mm, vias 2 -> 0
- net D13: track 117.4 -> 0.00 mm
- net A11: track 115.9 -> 0.00 mm, vias 1 -> 0
- net D6: track 113.6 -> 0.00 mm, vias 2 -> 0
- net A8: track 113.4 -> 0.00 mm, vias 1 -> 0
- net +BATT: track 113.2 -> 0.00 mm, vias 3 -> 0
- net D35: track 110.1 -> 0.00 mm, vias 1 -> 0
- net A6: track 109.7 -> 0.00 mm, vias 1 -> 0
- net A2: track 109.6 -> 0.00 mm, vias 2 -> 0
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- removed copper zone on B.Cu, net GND
- removed copper zone on F.Cu, net GND
Other:
- board size 100 x 100 mm -> 131.5 x 159.4 mm
- board text removed: "0"
- board text removed: "1"
- board text removed: "2"
- board text removed: "220R"
- board text removed: "3"
- board text removed: "3V"
- board text removed: "3V3"
- board text removed: "3V3 5V"
- board text removed: "4"
- board text removed: "470"
- board text removed: "5"
- board text removed: "5V"
- board text removed: "5V USB"
- board text removed: "6"
- board text removed: "7"
- board text removed: "A0"
- board text removed: "A1"
- board text removed: "A10"
- board text removed: "A11"
- board text removed: "A12"
- board text removed: "A13"
- board text removed: "A14"
- board text removed: "A15"
- board text removed: "A2"
- board text removed: "A3"
- board text removed: "A4"
- board text removed: "A5"
- board text removed: "A6"
- board text removed: "A7"
- board text removed: "A8"
- board text removed: "A9"
- board text removed: "AUD"
- board text removed: "CARTRIDGE PORT ADAPTER"
- board text removed: "CLK"
- board text removed: "CLK0"
- board text removed: "CLK1"
- board text removed: "CLK2"
- board text removed: "CLKGEN"
- board text removed: "CS"
- board text removed: "CS2"
- board text removed: "D0"
- board text removed: "D1"
- board text removed: "D10"
- board text removed: "D11"
- board text removed: "D12"
- board text removed: "D13"
- board text removed: "D14"
- board text removed: "D15"
- board text removed: "D16"
- board text removed: "D17"
- board text removed: "D18"
- board text removed: "D19"
- board text removed: "D2"
- board text removed: "D20"
- board text removed: "D21"
- board text removed: "D22"
- board text removed: "D23"
- board text removed: "D24"
- board text removed: "D25"
- board text removed: "D26"
- board text removed: "D27"
- board text removed: "D28"
- board text removed: "D29"
- board text removed: "D3"
- board text removed: "D30"
- board text removed: "D31"
- board text removed: "D32"
- board text removed: "D33"
- board text removed: "D34"
- board text removed: "D35"
- board text removed: "D36"
- board text removed: "D37"
- board text removed: "D38"
- board text removed: "D39"
- board text removed: "D4"
- board text removed: "D40"
- board text removed: "D41"
- board text removed: "D42"
- board text removed: "D43"
- board text removed: "D44"
- board text removed: "D45"
- board text removed: "D46"
- board text removed: "D47"
- board text removed: "D48"
- board text removed: "D49"
- board text removed: "D5"
- board text removed: "D50"
- board text removed: "D51"
- board text removed: "D52"
- board text removed: "D53"
- board text removed: "D6"
- board text removed: "D7"
- board text removed: "D8"
- board text removed: "D9"
- board text removed: "EXP1"
- board text removed: "EXP2"
- board text removed: "GAMEBOY SLOT"
- board text removed: "GND"
- board text removed: "HW5"
- board text removed: "I2C"
- board text removed: "JLCJLCJLCJLC"
- board text removed: "MISO"
- board text removed: "MKS MINI12864 V3"
- board text removed: "MOSI"
- board text removed: "NEOPIXEL"
- board text removed: "OFF"
- board text removed: "ON"
- board text removed: "ON OFF"
- board text removed: "PORT A"
- board text removed: "PORT C"
- board text removed: "PORT E"
- board text removed: "PORT F"
- board text removed: "PORT G"
- board text removed: "PORT H"
- board text removed: "PORT J"
- board text removed: "PORT K"
- board text removed: "PORT L"
- board text removed: "POWER"
- board text removed: "RD"
- board text removed: "RESET"
- board text removed: "REV${REVISION}"
- board text removed: "RST"
- board text removed: "RTC"
- board text removed: "RTC BATTERY"
- board text removed: "SCK"
- board text removed: "SCL"
- board text removed: "SDA"
- board text removed: "SPI"
- board text removed: "SS"
- board text removed: "STATUS LED"
- board text removed: "VCC"
- board text removed: "VOLTAGE"
- board text removed: "VSELECT"
- board text removed: "WR"
- board text removed: "uF"
