File: hardware/main_pcb_hw5/main_pcb_hw5.kicad_sch (KiCad schematic)
At the start: 25 parts, among them J1 MEGA BOTTOM, J10 GBA_Slot, J3 CART SLOT TOP ROW, J4 CART SLOT FRONT ROW, J6 5V USB, J7 Conn_01x07, J8 EXP2, J9 EXP1, M2_1 Screw_Terminal_01x01, M2_2 Screw_Terminal_01x01, M2_3 Screw_Terminal_01x01, M2_4 Screw_Terminal_01x01, M2_5 Screw_Terminal_01x01, M2_6 Screw_Terminal_01x01, M2_7 Screw_Terminal_01x01, M2_8 Screw_Terminal_01x01, M2_9 Screw_Terminal_01x01, SW1 VOLTAGE, SW2 POWER, U2 DS3231MZ

Commit message: cliche commit summary goes here
Parts:
- removed D1: LED, LED_THT:LED_D3.0mm, symbol Device:LED
- removed J10: GBA_Slot, symbol !OSCR:GBA_Slot
- removed J3: CART SLOT TOP ROW, !OSCR:Cartridge_Port_Adapter-Back, symbol Connector_Generic:Conn_01x38
- removed J4: CART SLOT FRONT ROW, !OSCR:Cartridge_Port_Adapter-Front, symbol Connector_Generic:Conn_01x36
- removed J6: 5V USB, Connector_PinHeader_2.54mm:PinHeader_1x01_P2.54mm_Vertical, symbol Connector_Generic:Conn_01x01
- removed J7: Conn_01x07, !OSCR:Clock_Generator_Header, symbol Connector_Generic:Conn_01x07
- removed J8: EXP2, !OSCR:LCD_Header, symbol Connector_Generic:Conn_02x05_Odd_Even
- removed J9: EXP1, !OSCR:LCD_Header, symbol Connector_Generic:Conn_02x05_Odd_Even
- removed M2_5, M2_6, M2_7, M2_8, M2_9: Screw_Terminal_01x01, symbol Connector:Screw_Terminal_01x01
- removed SW1: VOLTAGE, !OSCR:Power_Switch, symbol Switch:SW_SPDT
- removed SW2: POWER, !OSCR:Power_Switch, symbol Switch:SW_SPDT
- removed U2: DS3231MZ, Package_SO:SOIC-8_3.9x4.9mm_P1.27mm, symbol Timer_RTC:DS3231MZ
- added C1, C2, C28, C29, C3, C4, C5: 100nF, Capacitor_SMD:C_0805_2012Metric, symbol Device:C
- added C10, C11, C8, C9: 10uF, Capacitor_SMD:C_0805_2012Metric, symbol Device:C_Small
- added C12, C14, C18, C20, C22, C30: 1uF, Capacitor_SMD:C_0805_2012Metric, symbol Device:C_Small
- added C13, C16, C19, C21, C24, C31, C7: 100nF, Capacitor_SMD:C_0805_2012Metric, symbol Device:C_Small
- added C15, C17: 100nf, Capacitor_SMD:C_0805_2012Metric, symbol Device:C_Small
- added C23, C27: 0.1u, Capacitor_SMD:C_0805_2012Metric, symbol Device:C
- added C25, C26: 10uf, Capacitor_SMD:C_0805_2012Metric, symbol Device:C_Small
- added C34: 10u, Capacitor_SMD:C_0805_2012Metric, symbol Device:C
- added C35, C37: 22uf, Capacitor_SMD:C_0805_2012Metric, symbol Device:C_Polarized_Small_US
- added C39: C_Small_0.1uf, Capacitor_SMD:C_0805_2012Metric, symbol Device:C_Small
- added C6: 10uF, Capacitor_SMD:C_0805_2012Metric, symbol Device:C
- added Card1: TF PUSH, !MiniReader:TF-SMD_TF-PUSH, symbol !MiniReader:TFPUSH
- added D1, D11, D13, D14, D16, D18, D2, D20, D21, D23, D25, D26, D29, D3, D31, D33, D4, D7, D9: 1N4148W, Diode_SMD:D_SOD-123, symbol Diode:1N4148
- added D10, D12, D15, D17, D19, D22, D24, D27, D28, D5, D6, D8: SK6812MINI, !MiniReader:LED_SK6812MINI_PLCC4_3.5x3.5mm_P1.75mm, symbol LED:SK6812MINI
- added F1: MF-NSMF150-2, Fuse:Fuse_1206_3216Metric, symbol Device:Polyfuse
- added J1: Conn_01x03_Female, Connector_PinSocket_2.54mm:PinSocket_1x03_P2.54mm_Vertical, symbol LeChiffre-rescue:Conn_01x03_Female-Connector
- added J10, J11, J12, J7, J8, J9: SHOUHANTYPE-C16PIN2MD-073, !MiniReader:USB-C-SMD_TYPE-C-6PIN-2MD-073, symbol !MiniReader:TYPE-C16PIN2MD(073)
- added J14: Conn_01x09, Connector_PinHeader_1.00mm:PinHeader_1x09_P1.00mm_Vertical, symbol Connector_Generic:Conn_01x09
- added J3: Conn_02x36, !MiniReader:Secondary_Board_Connector, symbol Connector_Generic:Conn_02x36_Top_Bottom
- added J4: 5V USB, TestPoint:TestPoint_Pad_D2.0mm, symbol Connector_Generic:Conn_01x01
- added J5, J6: Conn_01x05, Connector_PinHeader_1.00mm:PinHeader_1x05_P1.00mm_Vertical, symbol Connector_Generic:Conn_01x05
- added JP1: Jumper_2_Open, Jumper:SolderJumper-2_P1.3mm_Open_TrianglePad1.0x1.5mm, symbol Jumper:Jumper_2_Open
- added L1: 60R@100MHz, Inductor_SMD:L_1206_3216Metric, symbol Unified-Daughterboard-rescue:L_Core_Ferrite-Device
- added R10, R11, R12, R13, R14, R3, R4, R5, R6, R7, R8, R9: 10K, Resistor_SMD:R_0805_2012Metric, symbol Device:R_Small
- added R15, R16, R17, R18: 3.3K, Resistor_SMD:R_0805_2012Metric, symbol Device:R_Small
- added R2: 560R, Resistor_SMD:R_0805_2012Metric, symbol Device:R
- added SW1: up, MX_Hotswap:MX-Hotswap-1U, symbol Switch:SW_Push
- added SW10, SW12, SW14, SW16, SW21: SKQGABE010, !MiniReader:SW-SMD_4P-L4.5-W4.5-P3.00-LS6.8, symbol !MiniReader:TSC015A05026A
- added SW11: b, MX_Hotswap:MX-Hotswap-1U, symbol Switch:SW_Push
- added SW13: c, MX_Hotswap:MX-Hotswap-1U, symbol Switch:SW_Push
- added SW15: d, MX_Hotswap:MX-Hotswap-1U, symbol Switch:SW_Push
- added SW17: l1, MX_Hotswap:MX-Hotswap-1U, symbol Switch:SW_Push
- added SW19: r1, MX_Hotswap:MX-Hotswap-1U, symbol Switch:SW_Push
- added SW2: l2h, MX_Hotswap:MX-Hotswap-1U, symbol Switch:SW_Push
- added SW22: Rotary_Encoder_Switch, !MiniReader:RotaryEncoder_EC11_no_mp, symbol LeChiffre-rescue:Rotary_Encoder_Switch-Device
- added SW3: down, MX_Hotswap:MX-Hotswap-1U, symbol Switch:SW_Push
- added SW4: l2l, MX_Hotswap:MX-Hotswap-1U, symbol Switch:SW_Push
- added SW5: left, MX_Hotswap:MX-Hotswap-1U, symbol Switch:SW_Push
- added SW6: r2h, MX_Hotswap:MX-Hotswap-1U, symbol Switch:SW_Push
- added SW7: right, MX_Hotswap:MX-Hotswap-1U, symbol Switch:SW_Push
- added SW8: r2l, MX_Hotswap:MX-Hotswap-1U, symbol Switch:SW_Push
- added SW9: a, MX_Hotswap:MX-Hotswap-1U, symbol Switch:SW_Push
- added U1: STM32F072CBT6, Package_QFP:LQFP-48_7x7mm_P0.5mm, symbol MCU_ST_STM32F0:STM32F072CBTx
- added U10: UZ1085L-33-TN3-R, Package_TO_SOT_SMD:TO-252-2, symbol Regulator_Linear:AZ1117-3.3
- added U11: DS1307DTR(XBLW), Package_SO:SOIC-8_3.9x4.9mm_P1.27mm, symbol Timer_RTC:DS3231MZ
- added U12: snesCIC PIC12F629T-E/MF1, Package_DFN_QFN:DFN-8-1EP_4x4mm_P0.8mm_EP2.39x2.21mm, symbol Connector_Generic_MountingPin:Conn_02x04_Counter_Clockwise_MountingPin
- added U13: 74LVC125APW,118, !MiniReader:TSSOP-14_L5.0-W4.4-P0.65-LS6.4-BL, symbol !MiniReader:74LVC125APW,118
- added U2: SL2.1A, Package_SO:SOIC-16_4.55x10.3mm_P1.27mm, symbol !MiniReader:SL2.1A
- added U3: SL2.1A, Package_SO:SOIC-16_4.55x10.3mm_P1.27mm, symbol SL2.1A:SL2.1A
- added U4, U5, U6, U7, U8: SMAJ8.0CA-TP, Diode_SMD:D_SMA, symbol Diode:SZESD9B5.0ST5G
- added U9: TPS2113PW, Package_SO:TSSOP-8_4.4x3mm_P0.65mm, symbol Added:TPS2113PW
- added Y1, Y2: 12mhz, Crystal:Crystal_HC49-4H_Vertical, symbol Device:Crystal
- added Y3: 32.768mhz, Crystal:Crystal_HC49-4H_Vertical, symbol Device:Crystal
- C36: renamed from C1; footprint Capacitor_THT:CP_Radial_D8.0mm_P3.50mm -> Capacitor_Tantalum_SMD:CP_EIA-7343-31_Kemet-D
- C38: renamed from C5; footprint Capacitor_SMD:C_0402_1005Metric_Pad0.74x0.62mm_HandSolder -> Capacitor_SMD:C_0805_2012Metric
- J2: renamed from J1; footprint !OSCR:MEGA2560_PRO_MINI -> !MiniReader:MEGA2560_PRO_EMBED_SMD
- M2_1, M2_2, M2_3, M2_4: footprint (none) -> MountingHole:MountingHole_2.2mm_M2_ISO7380_Pad
- R1: value 220R -> 10k; footprint Resistor_THT:R_Axial_DIN0207_L6.3mm_D2.5mm_P10.16mm_Horizontal -> Resistor_SMD:R_0805_2012Metric
Connections:
- net VBUS is gone; now on net +5V: C38.1
- net +3V3: now also C1.1, C2.1, C23.2, C3.1, C37.1, C4.1, C5.1, C6.1, Card1.4 (VDD), J14.6 (Pin_6), SW21.1, U1.1 (VBAT), U1.24 (VDD), U1.36 (VDDIO2), U1.48 (VDD), U1.9 (VDDA), U10.2 (VO), U13.14 (VCC), U9.8 (IN1)
- net +5V: now also C12.2, C13.2, C14.2, C15.1, C16.2, C17.1, C18.2, C19.2, C20.2, C21.2, C22.2, C24.2, C25.2, C26.2, C27.1, C30.2, C31.2, C35.1, D10.4 (VDD), D12.4 (VDD), D15.4 (VDD), D17.4 (VDD), D19.4 (VDD), D22.4 (VDD), D24.4 (VDD), D27.4 (VDD), D28.4 (VDD), D5.4 (VDD), D6.4 (VDD), D8.4 (VDD), F1.1, J1.3 (Pin_1), J10.11 (VBUS), J10.2 (VBUS), J11.11 (VBUS), J11.2 (VBUS), J12.11 (VBUS), J12.2 (VBUS), J5.5 (Pin_5), J6.5 (Pin_5), J7.11 (VBUS), J7.2 (VBUS), J8.11 (VBUS), J8.2 (VBUS), J9.11 (VBUS), J9.2 (VBUS), U10.3 (VI), U11.8 (VCC), U2.11 (VCC5V), U3.11 (VCC5V), U4.2 (A2), U9.6 (IN2)
- net +BATT: now also U11.3 (VBAT)
- net A0: now also J3.6 (Pin_6)
- net A1: now also J3.16 (Pin_16)
- net A10: now also J3.13 (Pin_13), J3.59 (Pin_59)
- net A11: now also J3.12 (Pin_12), J3.60 (Pin_60)
- net A12: now also J3.11 (Pin_11), J3.35 (Pin_35)
- net A13: now also J3.10 (Pin_10), J3.34 (Pin_34)
- net A14: now also J3.33 (Pin_33), J3.9 (Pin_9)
- net A15: now also D6.3 (DIN), J3.32 (Pin_32), J3.8 (Pin_8), JP1.1 (A), U1.38 (PA15)
- net A2: now also J3.22 (Pin_22)
- net A3: now also J3.23 (Pin_23)
- net A4: now also J3.24 (Pin_24)
- net A5: now also J3.48 (Pin_48)
- net A6: now also J3.42 (Pin_42)
- net A7: now also J3.41 (Pin_41)
- net A8: now also D1.2 (A), D11.2 (A), D14.2 (A), D18.2 (A), D21.2 (A), D25.2 (A), D29.2 (A), D3.2 (A), D31.2 (A), D7.2 (A), J3.15 (Pin_15), J3.57 (Pin_57), U1.29 (PA8)
- net A9: now also J3.14 (Pin_14), J3.58 (Pin_58)
- net CLK0: now also J3.5 (Pin_5)
- net CLK1: now also J3.1 (Pin_1)
- net CLK2: now also J3.67 (Pin_67), U12.2 (Pin_2)
- net D0: now also J3.61 (Pin_61)
- net D1: now also J3.66 (Pin_66)
- net D14: now also J3.3 (Pin_3)
- net D15: now also J3.2 (Pin_2)
- net D16: now also J3.20 (Pin_20)
- net D17: now also J3.21 (Pin_21)
- net D2: now also J3.72 (Pin_72)
- net D20: now also U11.5 (SDA)
- net D21: now also U11.6 (SCL)
- net D22: now also J3.26 (Pin_26)
- net D23: now also J3.27 (Pin_27)
- net D24: now also J3.29 (Pin_29)
- net D25: now also J3.28 (Pin_28)
- net D26: now also J3.30 (Pin_30)
- net D27: now also J3.31 (Pin_31)
- net D28: now also J3.7 (Pin_7)
- net D29: now also J3.4 (Pin_4)
- net D3: now also J3.36 (Pin_36)
- net D30: now also J3.47 (Pin_47)
- net D31: now also J3.46 (Pin_46)
- net D32: now also J3.45 (Pin_45)
- net D33: now also J3.44 (Pin_44)
- net D34: now also J3.43 (Pin_43)
- net D35: now also J3.49 (Pin_49)
- net D36: now also J3.65 (Pin_65)
- net D37: now also J3.64 (Pin_64)
- net D38: now also U9.3 (VSNS); no longer R1.2
- net D4: now also J3.62 (Pin_62)
- net D40: now also J3.37 (Pin_37), U12.4 (Pin_4)
- net D41: now also J3.38 (Pin_38), U12.3 (Pin_3)
- net D42: now also J3.25 (Pin_25)
- net D43: now also J3.50 (Pin_50)
- net D44: now also J3.51 (Pin_51)
- net D45: now also J3.52 (Pin_52)
- net D46: now also J3.53 (Pin_53)
- net D47: now also J3.54 (Pin_54)
- net D48: now also J3.55 (Pin_55)
- net D49: now also J3.56 (Pin_56)
- net D5: now also J3.68 (Pin_68)
- net D50: now also U13.11 (4Y); no longer J2.78 (D50)
- net D51: now also U13.3 (1Y); no longer J2.77 (D51)
- net D52: now also U13.6 (2Y); no longer J2.80 (D52)
- net D53: now also U13.8 (3Y); no longer J2.79 (D53)
- net D6: now also J3.19 (Pin_19)
- net D7: now also J3.18 (Pin_18)
- net D8: now also J3.17 (Pin_17)
- net D9: now also J3.70 (Pin_70)
- net GND: now also R1.2, C1.2, C10.2, C11.1, C12.1, C13.1, C14.1, C15.2, C16.1, C17.2, C18.1, C19.1, C2.2, C20.1, C21.1, C22.1, C23.1, C24.1, C25.1, C26.1, C27.2, C28.2, C29.2, C3.2, C30.1, C31.1, C34.2, C35.2, C37.2, C39.2, C4.2, C5.2, C6.2, C7.2, C8.2, C9.1, Card1.10, Card1.11, Card1.12, Card1.13, Card1.6 (VSS), D10.2 (VSS), D12.2 (VSS), D15.2 (VSS), D17.2 (VSS), D19.2 (VSS), D22.2 (VSS), D24.2 (VSS), D27.2 (VSS), D28.2 (VSS), D5.2 (VSS), D6.2 (VSS), D8.2 (VSS), J1.1 (Pin_3), J10.1 (GND), J10.12 (GND), J10.13 (SHELL), J10.14 (SHELL), J11.1 (GND), J11.12 (GND), J11.13 (SHELL), J11.14 (SHELL), J12.1 (GND), J12.12 (GND), J12.13 (SHELL), J12.14 (SHELL), J14.4 (Pin_4), J3.40 (Pin_40), J3.71 (Pin_71), J5.1 (Pin_1), J5.2 (Pin_2), J6.1 (Pin_1), J6.2 (Pin_2), J7.1 (GND), J7.12 (GND), J7.13 (SHELL), J7.14 (SHELL), J8.1 (GND), J8.12 (GND), J8.13 (SHELL), J8.14 (SHELL), J9.1 (GND), J9.12 (GND), J9.13 (SHELL), J9.14 (SHELL), L1.1, L1.2, R10.1, R11.1, R12.1, R13.1, R14.1, R2.1, R3.1, R4.1, R5.1, R6.1, R7.1, R8.1, R9.1, SW22.C, U1.23 (VSS), U1.35 (VSS), U1.47 (VSS), U1.8 (VSSA), U10.1 (GND), U11.4 (GND), U12.8 (Pin_8), U12.9 (MountPin), U13.1 (1OE), U13.10 (3OE), U13.13 (4OE), U13.4 (2OE), U13.7 (GND), U2.12 (GND), U3.12 (GND), U4.1 (A1), U5.1 (A1), U6.1 (A1), U7.1 (A1), U8.1 (A1), U9.2 (~{EN}), U9.5 (GND)
- net VCC: now also C34.1, C39.1, J3.63 (Pin_63), J3.69 (Pin_69), U12.1 (Pin_1), U9.7 (OUT)
- net BOOT0: now reaches R1.1
- net BOOT0: now also SW21.4, U1.44 (BOOT0)
- net D10: no longer names the net of J2.21 (D10)
- net D11: no longer names the net of J2.22 (D11)
- net D12: no longer names the net of J2.19 (D12)
- net D13: no longer names the net of J2.20 (D13)
- net D18: no longer names the net of J2.13 (D18)
- net D19: no longer names the net of J2.14 (D19)
- net D39: no longer names the net of J2.52 (D39)
- new net: J9.10 (CC2), R7.2
- new net: J9.4 (CC1), R8.2
- new net: D10.1 (DOUT), D15.3 (DIN), JP1.2 (B)
- new net: D10.3 (DIN), D6.1 (DOUT)
- new net: J8.10 (CC2), R5.2
- new net: J8.4 (CC1), R6.2
- new net: D13.1 (K), SW8.1
- new net: Card1.1 (DAT2), J14.9 (Pin_9)
- new net: Card1.2 (CD/DAT3), J14.8 (Pin_8), R16.1
- new net: Card1.3 (CMD), J14.7 (Pin_7), R17.1
- new net: Card1.5 (CLX), J14.5 (Pin_5), R18.1
- new net: Card1.7 (DAT0), J14.3 (Pin_3), R15.2
- new net: Card1.8 (DAT1), J14.2 (Pin_2)
- new net: Card1.9 (CD), J14.1 (Pin_1)
- new net: J10.10 (CC2), R9.2
- new net: R2.2, U9.4 (ILIM)
- new net: D5.1 (DOUT), J1.2 (Pin_2)
- new net: C10.1, U3.13 (VDD3)
- new net: C11.2, U3.14 (VDD18)
- new net: U3.15 (XOUT), U3.16 (XIN), Y2.1, Y2.2
- new net: J11.4 (CC1), R12.2
- new net: D3.1 (K), SW3.1
- new net: D18.1 (K), SW11.1
- new net: D20.1 (K), SW12.1
- new net: D2.1 (K), SW2.1
- new net: U11.2 (x2), Y3.1
- new net: U11.1 (x1), Y3.2
- new net: D16.1 (K), SW10.1
- new net: D21.1 (K), SW13.1
- new net: D26.1 (K), SW16.1
- new net: D4.1 (K), SW4.1
- new net: D31.1 (K), SW19.1
- new net: D12.1 (DOUT), D8.3 (DIN)
- new net: D12.3 (DIN), D17.1 (DOUT)
- new net: D29.1 (K), SW17.1
- new net: R16.2, U13.9 (3A)
- new net: D1.1 (K), SW1.1
- new net: J10.4 (CC1), R10.2
- new net: D7.1 (K), SW5.1
- new net: D19.1 (DOUT), D24.3 (DIN)
- new net: D15.1 (DOUT), D19.3 (DIN)
- new net: J12.4 (CC1), R14.2
- new net: R17.2, U13.2 (1A)
- new net: C8.1, U2.13 (VDD3)
- new net: C9.2, U2.14 (VDD18)
- new net: U2.15 (XOUT), U2.16 (XIN), Y1.1, Y1.2
- new net: D11.1 (K), SW7.1
- new net: D9.1 (K), SW6.1
- new net: D25.1 (K), SW15.1
- new net: D23.1 (K), SW14.1
- new net: J11.10 (CC2), R11.2
- new net: D33.1 (K), SW22.S2
- new net: R15.1, U13.12 (4A)
- new net: J12.10 (CC2), R13.2
- new net: D27.3 (DIN), D28.1 (DOUT)
- new net: D24.1 (DOUT), D28.3 (DIN)
- new net: J7.10 (CC2), R3.2
- new net: J7.4 (CC1), R4.2
- new net: R18.2, U13.5 (2A)
- new net: D14.1 (K), SW9.1
- new net: D17.3 (DIN), D22.1 (DOUT)
- new net: D5.3 (DIN), D8.1 (DOUT)
- new net: D22.3 (DIN), D27.1 (DOUT)
- new net +12V: J3.39 (Pin_39)
- new net +5.0V: F1.2, J4.1 (Pin_1)
- new net CIC DATA 0: U12.7 (Pin_7)
- new net CIC DATA 1: U12.6 (Pin_6)
- new net CIC RESET: U12.5 (Pin_5)
- new net D+: J5.3 (Pin_3), U2.10 (UDP), U5.2 (A2)
- new net D-: J5.4 (Pin_4), U2.9 (UDM), U6.2 (A2)
- new net D1+: J7.5 (DN2), J7.6 (DP1), J7.8 (DP2), U2.8 (DP1)
- new net D1-: J7.7 (DN1), U2.7 (DM1)
- new net D2+: J8.5 (DN2), J8.6 (DP1), J8.7 (DN1), J8.8 (DP2), U2.5 (DM2), U2.6 (DP2)
- new net D3+: J9.5 (DN2), J9.6 (DP1), J9.7 (DN1), J9.8 (DP2), U2.3 (DM3), U2.4 (DP3)
- new net D4+: J10.5 (DN2), J10.6 (DP1), J10.7 (DN1), J10.8 (DP2), U2.1 (DM4), U2.2 (DP4)
- new net D5+: J11.5 (DN2), J11.6 (DP1), J11.7 (DN1), J11.8 (DP2), U3.7 (DM1), U3.8 (DP1)
- new net D6+: J12.5 (DN2), J12.6 (DP1), J12.7 (DN1), J12.8 (DP2), U3.5 (DM2), U3.6 (DP2)
- new net D7+: U1.33 (PA12), U3.4 (DP3)
- new net D7-: U1.32 (PA11), U3.3 (DM3)
- new net DA+: J6.3 (Pin_3), U3.10 (UDP), U8.2 (A2)
- new net DA-: J6.4 (Pin_4), U3.9 (UDM), U7.2 (A2)
- new net EncA: C29.1, SW22.A, U1.40 (PB4)
- new net EncB: C28.1, SW22.B, U1.41 (PB5)
- new net NRST: C7.1, U1.7 (NRST)
- new net col0: SW1.2, SW2.2, U1.22 (PB11)
- new net col1: SW3.2, SW4.2, U1.25 (PB12)
- new net col2: SW5.2, SW6.2, U1.26 (PB13)
- new net col3: SW7.2, SW8.2, U1.27 (PB14)
- new net col4: SW10.4, SW9.2, U1.28 (PB15)
- new net col5: SW11.2, SW12.4, SW22.S1, U1.2 (PC13)
- new net col6: SW13.2, SW14.4, U1.3 (PC14)
- new net col7: SW15.2, SW16.4, U1.4 (PC15)
- new net col8: SW17.2, U1.5 (PF0)
- new net col9: SW19.2, U1.6 (PF1)
- new net row1: D13.2 (A), D16.2 (A), D2.2 (A), D20.2 (A), D23.2 (A), D26.2 (A), D33.2 (A), D4.2 (A), D9.2 (A), U1.21 (PB10)
- no-connect marks 13 -> 60
Other:
- removed sheet Voltage Select
- note added: "1"
- note added: "2"
- note added: "3"
- note added: "4"
- note added: "5"
- note added: "6"
- note added: "Differntial pair ref: 2 layer PCB microstrip spacing: 0.127mm coplanar reference spacing: 0.127mm signal width: 0.25mm dielectric thickness: 1.6mm calculator: https://www.eeweb.com/tools/edge-coupled-microstrip-impedance/ https://resources.altium.com/p/routing-requirements-usb-20-2-layer-pcb"
- note added: "MCU"
- note added: "MCU pin mapping"
- note added: "MiniReader"
- note added: "NRST has internal pull up Hold high for normal operation"
- note added: "POWER MANAGEMENT"
- note added: "SD CARD"
- note added: "SL2.1A"
- note added: "USB OUT"
- note added: "USB Port Decoupling"
- note added: "a"
- note added: "apologises fur bad inglish and apoligis for bad circuit"
- note added: "b"
- note added: "button to pull boot0 high while reseting to activate DFU"
- note added: "c"
- note added: "d"
- note added: "d-down"
- note added: "d-left"
- note added: "d-right"
- note added: "d-up"
- note added: "https://github.com/sanni/cartreader/discussions/874"
- note added: "l1"
- note added: "l2-h"
- note added: "l2-l"
- note added: "r1"
- note added: "r2-h"
- note added: "r2-l"
- note added: "ugly shcematic"
- note removed: "GBA SLOT"
- note removed: "LCD MODULE"
- title: OSCR HW5 -> MiniReader X1
- moved on the sheet: BT1, C36, C38, J2A, J2B, J2C, M2_1, M2_2, M2_3, M2_4
