File: hardware/main_pcb_hw5/vselect.kicad_sch (KiCad schematic)
At the start: 5 parts, among them U1 TPS2113PW

Commit message: cliche commit summary goes here
Parts:
- C2, C3, C4: footprint Capacitor_SMD:C_0402_1005Metric_Pad0.74x0.62mm_HandSolder -> Capacitor_SMD:C_0805_2012Metric
- R2: footprint Resistor_SMD:R_0402_1005Metric_Pad0.72x0.64mm_HandSolder -> Resistor_SMD:R_0805_2012Metric
- U1: footprint Personal:Texas_Instruments-TPS2113PW-Level_A -> Package_SO:TSSOP-8_4.4x3mm_P0.65mm
